Commit message: world link

File: HW1/arm_description/urdf/arm.urdf.xacro (robot description, xacro)
@@ -4,4 +4,10 @@
     <color rgba="1 0 0 1"/>
   </material>
+  <link name="world"/>
+  <joint name="arm_base_joint" type="fixed">
+    <parent link="world"/>
+    <child link="base_link"/>
+    <origin rpy="0.0 0 0" xyz="0 0 0"/>
+  </joint>
   <link name="base_link">
     <visual>
@@ -347,5 +353,5 @@
     </inertial>
   </link>
-  <xacro:include filename="$(find arm_gazebo)/urdf/camera.xacro"/>
+  <xacro:include filename="$(find arm_gazebo)/urdf/cam_tot.xacro"/>
   <xacro:my_camera parent="base_link"/>
   <gazebo>
@@ -354,4 +360,5 @@
       <controller_manager_prefix_node_name>controller_manager</controller_manager_prefix_node_name>
     </plugin>
+    <static>true</static>
   </gazebo>
   <xacro:include filename="$(find arm_description)/urdf/arm_hardware_interface.xacro"/>
